Commit message: nav2 and kcvision map is loaded and localization successfull

File: src/kc_vision_description/urd/modules/camera.xacro (robot description, xacro)
@@ -12,5 +12,5 @@
       <origin xyz="6.45358e-18 0 -0.0175" rpy="3.14159 -0 0"/>
       <geometry>
-        <mesh filename="package://slambot_description/assets/camera_link.stl"/>
+        <mesh filename="package://kc_vision_description/assets/camera_link.stl"/>
       </geometry>
       <material name="camera_link_material">
@@ -21,5 +21,5 @@
       <origin xyz="6.45358e-18 0 -0.0175" rpy="3.14159 -0 0"/>
       <geometry>
-        <mesh filename="package://slambot_description/assets/camera_link.stl"/>
+        <mesh filename="package://kc_vision_description/assets/camera_link.stl"/>
       </geometry>
     </collision>

File: src/kc_vision_description/urd/modules/chassis_and_wheels.xacro (robot description, xacro)
@@ -20,5 +20,5 @@
       <origin xyz="0 0 0" rpy="0 -0 0"/>
       <geometry>
-        <mesh filename="package://slambot_description/assets/base_link.stl"/>
+        <mesh filename="package://kc_vision_description/assets/base_link.stl"/>
       </geometry>
       <material name="base_link_material">
@@ -44,5 +44,5 @@
       <origin xyz="0 0 0.032" rpy="-1.5708 -0 0"/>
       <geometry>
-        <mesh filename="package://slambot_description/assets/wheel_link.stl"/>
+        <mesh filename="package://kc_vision_description/assets/wheel_link.stl"/>
       </geometry>
       <material name="wheel_link_material">
@@ -76,5 +76,5 @@
       <origin xyz="0 0 -0.032" rpy="1.5708 -0 0"/>
       <geometry>
-        <mesh filename="package://slambot_description/assets/wheel_link.stl"/>
+        <mesh filename="package://kc_vision_description/assets/wheel_link.stl"/>
       </geometry>
       <material name="wheel_link_2_material">
@@ -108,5 +108,5 @@
       <origin xyz="0 0 -0.032" rpy="1.5708 -0 0"/>
       <geometry>
-        <mesh filename="package://slambot_description/assets/wheel_link.stl"/>
+        <mesh filename="package://kc_vision_description/assets/wheel_link.stl"/>
       </geometry>
       <material name="wheel_link_3_material">
@@ -140,5 +140,5 @@
       <origin xyz="0 0 0.032" rpy="-1.5708 -0 0"/>
       <geometry>
-        <mesh filename="package://slambot_description/assets/wheel_link.stl"/>
+        <mesh filename="package://kc_vision_description/assets/wheel_link.stl"/>
       </geometry>
       <material name="wheel_link_4_material">

File: src/kc_vision_description/urd/modules/lidar.xacro (robot description, xacro)
@@ -12,5 +12,5 @@
       <origin xyz="0 1.22465e-18 0" rpy="3.14159 -0 0"/>
       <geometry>
-        <mesh filename="package://slambot_description/assets/lidar_link.stl"/>
+        <mesh filename="package://kc_vision_description/assets/lidar_link.stl"/>
       </geometry>
       <material name="lidar_link_material">
@@ -21,5 +21,5 @@
       <origin xyz="0 1.22465e-18 0" rpy="3.14159 -0 0"/>
       <geometry>
-        <mesh filename="package://slambot_description/assets/lidar_link.stl"/>
+        <mesh filename="package://kc_vision_description/assets/lidar_link.stl"/>
       </geometry>
     </collision>

File: src/kc_vision_description/urd/modules/ros2_control_sim.xacro (robot description, xacro)
@@ -4,5 +4,5 @@
 <!-- WE WILL DO THIS SO THE ROBOTS KINEMATICS BEHAVIOUR IS AS CLOSE IN SIM AS POSSIBLE TO HOW IT BEHAVE IN REAL LIFE-->
 <!-- =============== DiffDrive (Using the ROS2_CONTROL diff-drive-controller!!)=============== -->
-    <ros2_control name="slambot" type="system">
+    <ros2_control name="kc_vision" type="system">
         <hardware>
             <plugin>gz_ros2_control/GazeboSimSystem</plugin>
@@ -35,5 +35,5 @@
             <remapping>diff_drive_controller/odom:=/odom</remapping> <!-- CRITICAL WE DO THIS - SEE BELOW FOR WHY-->
             </ros>
-            <parameters>$(find slambot_bringup)/config/slambot_controllers.yaml</parameters>
+            <parameters>$(find kc_vision_bringup)/config/kc_vision_controllers.yaml</parameters>
         </plugin>
     </gazebo>

File: src/kc_vision_description/urd/slambot.urdf.xacro (robot description, xacro)
@@ -18,5 +18,5 @@
     </xacro:unless>
     <!-- ... inside the launch file we then use commands such as this ...
-    xacro_file = os.path.join(get_package_share_directory('slambot_description'), 'urdf', 'slambot.urdf.xacro')
+    xacro_file = os.path.join(get_package_share_directory('kc_vision_description'), 'urdf', 'kc_vision.urdf.xacro')
     robot_description_config = Command(['xacro ', xacro_file, ' using_sim:=false'])
     params = {'robot_description': robot_description_config}

File: src/kc_vision_description/urd/xacro_properties/xacro_properties.xacro (robot description, xacro)
@@ -1,5 +1,5 @@
 <?xml version="1.0" ?>
 <robot xmlns:xacro="http://www.ros.org/wiki/xacro">
-  <xacro:property name="package_name" value="slambot_description" />
-  <xacro:property name="robot_name" value="slambot" />
+  <xacro:property name="package_name" value="kc_vision_description" />
+  <xacro:property name="robot_name" value="kc_vision" />
 </robot>
