Commit message: navigation is working in real.

File: src/kc_vision_description/urdf/modules/kc.xacro (robot description, xacro)
@@ -569,4 +569,5 @@
   <child link="front_right_rim_1"/>
   <axis xyz="0.0 1.0 0.0"/>
+  <mimic joint="rear_right_wheel_joint" multiplier="1.0" offset="0.0"/>
 </joint>
 <joint name="Rigid 17" type="fixed">
@@ -580,4 +581,5 @@
   <child link="front_left_rim_1"/>
   <axis xyz="0.0 1.0 0.0"/>
+  <mimic joint="rear_left_wheel_joint" multiplier="1.0" offset="0.0"/>
 </joint>
 <joint name="Rigid 19" type="fixed">

File: src/kc_vision_description/urdf/modules/ros2_control.xacro (robot description, xacro)
@@ -3,5 +3,6 @@
   <ros2_control name="SlambotReal" type="system">
     <hardware>
-      <plugin>slambot_hardware/SlambotHardwareInterface</plugin>
+      <plugin>kc_vision_hardware/KCVisionHardwareInterface</plugin>
+      <!-- <plugin>slambot_hardware/SlambotHardwareInterface</plugin> -->
     </hardware>
     <joint name="rear_left_wheel_joint">

File: src/kc_vision_description/urdf/modules/ros2_control_sim.xacro (robot description, xacro)
@@ -8,5 +8,5 @@
             <plugin>gz_ros2_control/GazeboSimSystem</plugin>
         </hardware>
-        <joint name="front_left_wheel_joint">
+        <!-- <joint name="front_left_wheel_joint">
             <command_interface name="velocity">
                 <param name="min">-10</param>
@@ -23,5 +23,5 @@
             <state_interface name="position"/>
             <state_interface name="velocity"/>
-        </joint>
+        </joint> -->
         <joint name="rear_left_wheel_joint">
             <command_interface name="velocity">

Commit message: slam and GPS based boustrophedon pattern done.

File: src/kc_vision_description/urdf/modules/kc.xacro (robot description, xacro)
@@ -569,5 +569,5 @@
   <child link="front_right_rim_1"/>
   <axis xyz="0.0 1.0 0.0"/>
-  <mimic joint="rear_right_wheel_joint" multiplier="1.0" offset="0.0"/>
+  <!-- <mimic joint="rear_right_wheel_joint" multiplier="1.0" offset="0.0"/> -->
 </joint>
 <joint name="Rigid 17" type="fixed">
@@ -581,5 +581,5 @@
   <child link="front_left_rim_1"/>
   <axis xyz="0.0 1.0 0.0"/>
-  <mimic joint="rear_left_wheel_joint" multiplier="1.0" offset="0.0"/>
+  <!-- <mimic joint="rear_left_wheel_joint" multiplier="1.0" offset="0.0"/> -->
 </joint>
 <joint name="Rigid 19" type="fixed">

File: src/kc_vision_description/urdf/modules/ros2_control_sim.xacro (robot description, xacro)
@@ -8,5 +8,5 @@
             <plugin>gz_ros2_control/GazeboSimSystem</plugin>
         </hardware>
-        <!-- <joint name="front_left_wheel_joint">
+        <joint name="front_left_wheel_joint">
             <command_interface name="velocity">
                 <param name="min">-10</param>
@@ -23,5 +23,5 @@
             <state_interface name="position"/>
             <state_interface name="velocity"/>
-        </joint> -->
+        </joint>
         <joint name="rear_left_wheel_joint">
             <command_interface name="velocity">
